File: TalkingClock.kicad_pcb (KiCad board)
At the start: 2 copper layers, 116 x 63.5 mm, 9 parts, among them J2 Micro_SD_Card_Det1, U1 AT42QT1010-TSHR, U2 E73-2G4M08S1C

Commit message: add things
Parts:
- removed J2: Micro_SD_Card_Det1, Connector_Card:microSD_HC_Molex_104031-0811
- JP2: moved to B.Cu
- moved BT1 27.0 mm to (165.1, 112.9)
- moved JP2 13.8 mm to (172.9, 106.5)
- moved C1 13.5 mm to (147.3, 110.3), turned to 180 degrees
- moved U1 11.3 mm to (147.3, 108.2)
- moved R1 6.50 mm to (146.3, 113.8)
Routing:
- net (no net): track 0.00 -> 8.65 mm, vias 0 -> 1
Other:
- board size 116 x 63.5 mm -> 112.9 x 57.5 mm
- board text added: "Flex"
